File: kicad/NanoV3.2.sch (KiCad schematic (older format))
At the start: 14 parts, among them IC2 LM1117IMPX-5.0, IC3 ATMEGA328P-AU, P1 CONN_01X03, SW1 RESET, Y1 16MHz

Commit message: added relay
Parts:
- added P2: OUT, symbol CONN_01X02
- added Q1: BC237, TO-92, symbol BC237
- added RL1: FINDER-40.31, symbol FINDER-40.31
- P1: value CONN_01X03 -> TTL
Connections:
- wire segments 59 -> 69
Other:
- note removed: "+5V AUTO SELECTOR"
Changed lines of the file:
@@
 LIBS:NanoV3.2
 LIBS:conn
-LIBS:NanoV3.2-cache
+LIBS:relays
+LIBS:transistors
 EELAYER 25 0
 EELAYER END
@@
 Text Notes 12300 9350 0    150  ~ 0
 ICSP
-Text Notes 7900 12450 0    150  ~ 0
-+5V AUTO SELECTOR
 $Comp
 L 0015_100NF_0603 C1
@@
 F 3 "" H 6400 10050 60  0001 C CNN
 	1    6400 10050
-	1    0    0    -1
-$EndComp
-$Comp
-L A3-FRAME-STANDARD FRAME1
-U 1 1 5A38BE68
-P 3500 12750
-F 0 "FRAME1" H 3490 12740 65  0001 L TNN
-F 1 "DNP" H 3490 12640 65  0001 L TNN
-F 2 "FRAME" H 3490 12540 65  0001 L TNN
-F 3 "" H 3500 12750 60  0001 C CNN
-	1    3500 12750
 	1    0    0    -1
 $EndComp
@@
 NoConn ~ 9100 6950
 NoConn ~ 9100 6850
-Wire Wire Line
-	6000 9850 6700 9850
-Wire Wire Line
-	6400 9750 6400 9950
-Wire Wire Line
-	6000 9950 6100 9950
-Wire Wire Line
-	6100 9950 6100 9850
-Connection ~ 6400 9850
-Connection ~ 6100 9850
-Wire Wire Line
-	5700 7550 7200 7550
-Wire Wire Line
-	7200 6950 6700 6950
-Wire Wire Line
-	6700 6950 6700 7650
-Wire Wire Line
-	6200 7650 6200 7850
-Wire Wire Line
-	5100 7650 6200 7650
-Wire Wire Line
-	6700 7650 7200 7650
-Wire Wire Line
-	5100 7650 5100 7750
-Connection ~ 6700 7550
-Connection ~ 5700 7550
-Connection ~ 5700 7650
-Wire Wire Line
-	12700 9750 13000 9750
-Wire Wire Line
-	13000 9750 13000 9550
-Wire Wire Line
-	6200 5550 6200 5450
-Wire Wire Line
-	7200 6850 5000 6850
-Wire Wire Line
-	5000 6850 5000 7050
-Wire Wire Line
-	5000 7350 5000 7450
-Wire Wire Line
-	6200 8150 6200 8350
-Wire Wire Line
-	5700 8150 5700 8250
-Wire Wire Line
-	5100 8250 6200 8250
-Wire Wire Line
-	5100 8250 5100 8050
-Connection ~ 6200 8250
-Connection ~ 5700 8250
-Wire Wire Line
-	12700 9950 13000 9950
-Wire Wire Line
-	13000 9950 13000 10150
-Wire Wire Line
-	5100 6150 4700 6150
-Wire Wire Line
-	5600 10550 5600 10250
-Wire Wire Line
-	7400 10550 7400 10450
-Wire Wire Line
-	6300 6550 6100 6550
-Wire Wire Line
-	6100 6550 6100 6650
-Wire Wire Line
-	7200 7050 7000 7050
-Wire Wire Line
-	7000 7050 7000 7450
-Wire Wire Line
-	6800 7350 7200 7350
-Wire Wire Line
-	7000 7450 7200 7450
-Connection ~ 7000 7350
-Wire Wire Line
-	6400 10450 6400 10250
-Wire Wire Line
-	9100 8250 9900 8250
-Wire Wire Line
-	9100 8150 9900 8150
-Wire Wire Line
-	13600 9850 12700 9850
-Wire Wire Line
-	9100 6350 9500 6350
-Wire Wire Line
-	11400 9750 12400 9750
-Wire Wire Line
-	9100 6250 9500 6250
-Wire Wire Line
-	11400 9850 12400 9850
-Wire Wire Line
-	6900 6450 6600 6450
-Wire Wire Line
-	7200 6550 6900 6550
-Wire Wire Line
-	6900 6550 6900 6450
-Wire Wire Line
-	6600 6650 7200 6650
-Wire Wire Line
-	7400 9850 7400 10150
-Wire Wire Line
-	7100 9850 7400 9850
-Wire Wire Line
-	11400 9950 12400 9950
-Wire Wire Line
-	5700 6150 6200 6150
-Wire Wire Line
-	6200 6150 6200 5950
-Wire Wire Line
-	7200 6150 6700 6150
-Wire Wire Line
-	10300 8150 11000 8150
-Wire Wire Line
-	4800 9750 4800 9850
-Wire Wire Line
-	4800 9850 5300 9850
-Wire Wire Line
-	9100 6150 9500 6150
 $Comp
 L CONN_01X03 P1
@@
 P 11200 8250
 F 0 "P1" H 11200 8450 50  0000 C CNN
-F 1 "CONN_01X03" V 11300 8250 50  0000 C CNN
+F 1 "TTL" V 11300 8250 50  0000 C CNN
 F 2 "Pin_Headers:Pin_Header_Straight_1x03" H 11200 8250 50  0001 C CNN
 F 3 "" H 11200 8250 50  0000 C CNN
@@
 Text Label 10500 8450 0    65   ~ 0
 RX
-Wire Wire Line
-	9900 8250 9900 8350
-Wire Wire Line
-	10300 8350 10700 8350
-Wire Wire Line
-	10700 8350 10700 8250
-Wire Wire Line
-	10700 8250 11000 8250
 $Comp
 L COM #M015
@@
 	1    0    0    -1
 $EndComp
-Wire Wire Line
-	5700 7250 5700 7850
 NoConn ~ 9100 6450
 Text Label 9100 6550 0    10   ~ 0
@@
 	1    0    0    -1
 $EndComp
+$Comp
+L FINDER-40.31 RL1
+U 1 1 5A3B4306
+P 13100 6850
+F 0 "RL1" H 13550 7000 50  0000 L CNN
+F 1 "FINDER-40.31" H 13550 6900 50  0000 L CNN
+F 2 "" H 13100 6850 50  0000 C CNN
+F 3 "" H 13100 6850 50  0000 C CNN
+	1    13100 6850
+	1    0    0    -1
+$EndComp
+$Comp
+L COM #M016
+U 1 1 5A3B4697
+P 12900 7350
+F 0 "#M016" H 12900 7350 45  0001 C CNN
+F 1 "COM" H 12900 7350 45  0001 C CNN
+F 2 "" H 12900 7350 60  0000 C CNN
+F 3 "" H 12900 7350 60  0000 C CNN
+	1    12900 7350
+	1    0    0    -1
+$EndComp
+$Comp
+L +5V #M017
+U 1 1 5A3B46CD
+P 12900 5950
+F 0 "#M017" H 12900 5950 45  0001 L BNN
+F 1 "+5V" H 12800 6050 45  0000 L BNN
+F 2 "" H 12900 5950 60  0000 C CNN
+F 3 "" H 12900 5950 60  0000 C CNN
+	1    12900 5950
+	1    0    0    -1
+$EndComp
+$Comp
+L BC237 Q1
+U 1 1 5A3B4AFF
+P 12800 6300
+F 0 "Q1" H 13000 6375 50  0000 L CNN
+F 1 "BC237" H 13000 6300 50  0000 L CNN
+F 2 "TO-92" H 13000 6225 50  0000 L CIN
+F 3 "" H 12800 6300 50  0000 L CNN
+	1    12800 6300
+	1    0    0    -1
+$EndComp
+Wire Wire Line
+	6000 9850 6700 9850
+Wire Wire Line
+	6400 9750 6400 9950
+Wire Wire Line
+	6000 9950 6100 9950
+Wire Wire Line
+	6100 9950 6100 9850
+Connection ~ 6400 9850
+Connection ~ 6100 9850
+Wire Wire Line
+	5700 7550 7200 7550
+Wire Wire Line
+	7200 6950 6700 6950
+Wire Wire Line
+	6700 6950 6700 7650
+Wire Wire Line
+	6200 7650 6200 7850
+Wire Wire Line
+	5100 7650 6200 7650
+Wire Wire Line
+	6700 7650 7200 7650
+Wire Wire Line
+	5100 7650 5100 7750
+Connection ~ 6700 7550
+Connection ~ 5700 7550
+Connection ~ 5700 7650
+Wire Wire Line
+	12700 9750 13000 9750
+Wire Wire Line
+	13000 9750 13000 9550
+Wire Wire Line
+	6200 5550 6200 5450
+Wire Wire Line
+	7200 6850 5000 6850
+Wire Wire Line
+	5000 6850 5000 7050
+Wire Wire Line
+	5000 7350 5000 7450
+Wire Wire Line
+	6200 8150 6200 8350
+Wire Wire Line
+	5700 8150 5700 8250
+Wire Wire Line
+	5100 8250 6200 8250
+Wire Wire Line
+	5100 8250 5100 8050
+Connection ~ 6200 8250
+Connection ~ 5700 8250
+Wire Wire Line
+	12700 9950 13000 9950
+Wire Wire Line
+	13000 9950 13000 10150
+Wire Wire Line
+	5100 6150 4700 6150
+Wire Wire Line
+	5600 10550 5600 10250
+Wire Wire Line
+	7400 10550 7400 10450
+Wire Wire Line
+	6300 6550 6100 6550
+Wire Wire Line
+	6100 6550 6100 6650
+Wire Wire Line
+	7200 7050 7000 7050
+Wire Wire Line
+	7000 7050 7000 7450
+Wire Wire Line
+	6800 7350 7200 7350
+Wire Wire Line
+	7000 7450 7200 7450
+Connection ~ 7000 7350
+Wire Wire Line
+	6400 10450 6400 10250
+Wire Wire Line
+	9100 8250 9900 8250
+Wire Wire Line
+	9100 8150 9900 8150
+Wire Wire Line
+	13600 9850 12700 9850
+Wire Wire Line
+	9100 6350 9500 6350
+Wire Wire Line
+	11400 9750 12400 9750
+Wire Wire Line
+	9100 6250 9500 6250
+Wire Wire Line
+	11400 9850 12400 9850
+Wire Wire Line
+	6900 6450 6600 6450
+Wire Wire Line
+	7200 6550 6900 6550
+Wire Wire Line
+	6900 6550 6900 6450
+Wire Wire Line
+	6600 6650 7200 6650
+Wire Wire Line
+	7400 9850 7400 10150
+Wire Wire Line
+	7100 9850 7400 9850
+Wire Wire Line
+	11400 9950 12400 9950
+Wire Wire Line
+	5700 6150 6200 6150
+Wire Wire Line
+	6200 6150 6200 5950
+Wire Wire Line
+	7200 6150 6700 6150
+Wire Wire Line
+	10300 8150 11000 8150
+Wire Wire Line
+	4800 9750 4800 9850
+Wire Wire Line
+	4800 9850 5300 9850
+Wire Wire Line
+	9100 6150 9500 6150
+Wire Wire Line
+	9900 8250 9900 8350
+Wire Wire Line
+	10300 8350 10700 8350
+Wire Wire Line
+	10700 8350 10700 8250
+Wire Wire Line
+	10700 8250 11000 8250
+Wire Wire Line
+	5700 7250 5700 7850
+Wire Wire Line
+	12900 7150 12900 7250
+Wire Wire Line
+	12900 6550 12900 6500
+Wire Wire Line
+	12900 6050 12900 6100
+Wire Wire Line
+	12600 6300 12350 6300
+Wire Wire Line
+	13200 6550 13200 6450
+$Comp
+L VIN #M018
+U 1 1 5A3B5FE9
+P 14050 6350
+F 0 "#M018" H 14050 6350 45  0001 L BNN
+F 1 "VIN" H 13970 6450 45  0000 L BNN
+F 2 "" H 14050 6350 60  0000 C CNN
+F 3 "" H 14050 6350 60  0000 C CNN
+	1    14050 6350
+	1    0    0    -1
+$EndComp
+Wire Wire Line
+	13200 6450 14050 6450
+$Comp
+L CONN_01X02 P2
+U 1 1 5A3B61A1
+P 14100 7300
+F 0 "P2" H 14100 7450 50  0000 C CNN
+F 1 "OUT" V 14200 7300 50  0000 C CNN
+F 2 "" H 14100 7300 50  0000 C CNN
+F 3 "" H 14100 7300 50  0000 C CNN
+	1    14100 7300
+	1    0    0    -1
+$EndComp
+Wire Wire Line
+	13300 7150 13300 7250
+Wire Wire Line
+	13300 7250 13900 7250
+$Comp
+L COM #M019
+U 1 1 5A3B62DB
+P 13900 7600
+F 0 "#M019" H 13900 7600 45  0001 C CNN
+F 1 "COM" H 13900 7600 45  0001 C CNN
+F 2 "" H 13900 7600 60  0000 C CNN
+F 3 "" H 13900 7600 60  0000 C CNN
+	1    13900 7600
+	1    0    0    -1
+$EndComp
+Wire Wire Line
+	13900 7500 13900 7350
+Text Label 12400 6300 0    60   ~ 0
+D2
+Wire Wire Line
+	9100 8050 9300 8050
+Text Label 9200 8050 0    60   ~ 0
+D2
+$Comp
+L A3-FRAME-STANDARD FRAME1
+U 1 1 5A38BE68
+P 3500 12750
+F 0 "FRAME1" H 3490 12740 65  0001 L TNN
+F 1 "DNP" H 3490 12640 65  0001 L TNN
+F 2 "FRAME" H 3490 12540 65  0001 L TNN
+F 3 "" H 3500 12750 60  0001 C CNN
+	1    3500 12750
+	1    0    0    -1
+$EndComp
