File: kicad/NanoV3.2.sch (KiCad schematic (older format))
At the start: 23 parts, among them IC2 LM1117IMPX-5.0, IC3 ATMEGA328P-AU, P1 TTL, P2 OUT, P3 INPUT, Q1 BC237, Y1 16MHz

Commit message: updated jumpper pad
Parts:
- JP1, JP2, JP3, JP4, JP5, JP6: footprint C0603-ROUND -> autoSwitch:SMD-Jummper
Changed lines of the file:
@@
 LIBS:transistors
 LIBS:finder-40
+LIBS:NanoV3.2-cache
 EELAYER 25 0
 EELAYER END
@@
 F 0 "JP1" H 9800 7900 45  0000 L BNN
 F 1 "Jumpper" H 9950 7850 45  0000 L BNN
-F 2 "C0603-ROUND" H 9500 7800 20  0001 C CNN
+F 2 "autoSwitch:SMD-Jummper" H 9500 7800 20  0001 C CNN
 F 3 "" H 9650 7850 60  0000 C CNN
 	1    9650 7850
@@
 F 0 "JP2" H 9800 7800 45  0000 L BNN
 F 1 "Jumpper" H 9950 7750 45  0000 L BNN
-F 2 "C0603-ROUND" H 9500 7700 20  0001 C CNN
+F 2 "autoSwitch:SMD-Jummper" H 9500 7700 20  0001 C CNN
 F 3 "" H 9650 7750 60  0000 C CNN
 	1    9650 7750
@@
 F 0 "JP3" H 9800 7700 45  0000 L BNN
 F 1 "Jumpper" H 9950 7650 45  0000 L BNN
-F 2 "C0603-ROUND" H 9500 7600 20  0001 C CNN
+F 2 "autoSwitch:SMD-Jummper" H 9500 7600 20  0001 C CNN
 F 3 "" H 9650 7650 60  0000 C CNN
 	1    9650 7650
@@
 F 0 "JP4" H 9800 7600 45  0000 L BNN
 F 1 "Jumpper" H 9950 7550 45  0000 L BNN
-F 2 "C0603-ROUND" H 9500 7500 20  0001 C CNN
+F 2 "autoSwitch:SMD-Jummper" H 9500 7500 20  0001 C CNN
 F 3 "" H 9650 7550 60  0000 C CNN
 	1    9650 7550
@@
 F 0 "JP5" H 9800 6700 45  0000 L BNN
 F 1 "Jumpper" H 9950 6650 45  0000 L BNN
-F 2 "C0603-ROUND" H 9500 6600 20  0001 C CNN
+F 2 "autoSwitch:SMD-Jummper" H 9500 6600 20  0001 C CNN
 F 3 "" H 9650 6650 60  0000 C CNN
 	1    9650 6650
@@
 F 0 "JP6" H 9800 6600 45  0000 L BNN
 F 1 "Jumpper" H 9950 6550 45  0000 L BNN
-F 2 "C0603-ROUND" H 9500 6500 20  0001 C CNN
+F 2 "autoSwitch:SMD-Jummper" H 9500 6500 20  0001 C CNN
 F 3 "" H 9650 6550 60  0000 C CNN
 	1    9650 6550

Commit message: updated RP1 network and crytal footprint
Parts:
- JP1, JP2, JP3, JP4, JP5, JP6: value Jumpper -> ~
- Y1: footprint RESONATOR -> autoSwitch:Crystal3215
Other:
- moved on the sheet: PWR56
Changed lines of the file:
@@
 L 0043_KPT-2012SGC PWR56
 U 1 1 5A38C570
-P 7400 10250
-F 0 "PWR56" V 7540 10070 70  0000 L BNN
-F 1 "Green" V 7625 10070 70  0000 L BNN
-F 2 "CHIPLED_0805" H 7390 10040 65  0001 L TNN
-F 3 "" H 7400 10250 60  0001 C CNN
-	1    7400 10250
+P 11100 6550
+F 0 "PWR56" V 11240 6370 70  0000 L BNN
+F 1 "Green" V 11325 6370 70  0000 L BNN
+F 2 "CHIPLED_0805" H 11090 6340 65  0001 L TNN
+F 3 "" H 11100 6550 60  0001 C CNN
+	1    11100 6550
 	1    0    0    -1
 $EndComp
 $Comp
 L 0005_064R_1K___CAY16-102J4LF RP1
-U 1 1 5A38C638
+U 3 1 5A38C638
 P 10100 8350
 F 0 "RP1" H 10000 8130 70  0000 L BNN
@@
 F 2 "CAY16" H 10090 8140 65  0001 L TNN
 F 3 "" H 10100 8350 60  0001 C CNN
-	1    10100 8350
+	3    10100 8350
 	1    0    0    -1
 $EndComp
@@
 $EndComp
 $Comp
-L 0005_064R_1K___CAY16-102J4LF RP1
-U 3 1 5A38C700
-P 6900 9850
-F 0 "RP1" H 6801 9730 70  0000 L BNN
-F 1 "1K" H 6801 9630 70  0000 L BNN
-F 2 "CAY16" H 6890 9640 65  0001 L TNN
-F 3 "" H 6900 9850 60  0001 C CNN
-	3    6900 9850
-	-1   0    0    1
-$EndComp
-$Comp
 L COM #U$01
 U 1 1 5A38CCDC
@@
 L COM #U$010
 U 1 1 5A38D95C
-P 7400 10650
-F 0 "#U$010" H 7450 10700 60  0001 C CNN
-F 1 "~" H 7400 10650 60  0001 C CNN
-F 2 "" H 7400 10650 60  0001 C CNN
-F 3 "" H 7400 10650 60  0001 C CNN
-	1    7400 10650
+P 11100 6950
+F 0 "#U$010" H 11150 7000 60  0001 C CNN
+F 1 "~" H 11100 6950 60  0001 C CNN
+F 2 "" H 11100 6950 60  0001 C CNN
+F 3 "" H 11100 6950 60  0001 C CNN
+	1    11100 6950
 	1    0    0    -1
 $EndComp
@@
 F 0 "Y1" H 6400 6730 70  0000 L BNN
 F 1 "16MHz" H 6400 6330 70  0000 L BNN
-F 2 "RESONATOR" H 6590 6340 65  0001 L TNN
+F 2 "autoSwitch:Crystal3215" H 6590 6340 65  0001 L TNN
 F 3 "" H 6600 6550 60  0001 C CNN
 	1    6600 6550
@@
 +5V
 Text Label 6000 9850 0    10   ~ 0
-+5V
-Text Label 6700 9850 2    10   ~ 0
 +5V
 Text Label 6400 9950 1    10   ~ 0
@@
 Text Label 7200 6650 2    10   ~ 0
 N$2
-Text Label 7400 10150 1    10   ~ 0
+Text Label 11100 6450 1    10   ~ 0
 N$3
-Text Label 7100 9850 0    10   ~ 0
+Text Label 10800 6150 0    10   ~ 0
 N$3
 Text Label 12400 9950 2    10   ~ 0
@@
 $EndComp
 Wire Wire Line
-	6000 9850 6700 9850
-Wire Wire Line
 	6400 9750 6400 9950
 Wire Wire Line
@@
 	5600 10550 5600 10250
 Wire Wire Line
-	7400 10550 7400 10450
+	11100 6850 11100 6750
 Wire Wire Line
 	6300 6550 6100 6550
@@
 	6600 6650 7200 6650
 Wire Wire Line
-	7400 9850 7400 10150
-Wire Wire Line
-	7100 9850 7400 9850
+	11100 6150 11100 6450
+Wire Wire Line
+	10800 6150 11100 6150
 Wire Wire Line
 	11400 9950 12400 9950
@@
 	4800 9850 5300 9850
 Wire Wire Line
-	9100 6150 9500 6150
+	9100 6150 10400 6150
 Wire Wire Line
 	9900 8250 9900 8350
@@
 P 9650 7850
 F 0 "JP1" H 9800 7900 45  0000 L BNN
-F 1 "Jumpper" H 9950 7850 45  0000 L BNN
+F 1 "~" H 9950 7850 45  0000 L BNN
 F 2 "autoSwitch:SMD-Jummper" H 9500 7800 20  0001 C CNN
 F 3 "" H 9650 7850 60  0000 C CNN
@@
 P 9650 7750
 F 0 "JP2" H 9800 7800 45  0000 L BNN
-F 1 "Jumpper" H 9950 7750 45  0000 L BNN
+F 1 "~" H 9950 7750 45  0000 L BNN
 F 2 "autoSwitch:SMD-Jummper" H 9500 7700 20  0001 C CNN
 F 3 "" H 9650 7750 60  0000 C CNN
@@
 P 9650 7650
 F 0 "JP3" H 9800 7700 45  0000 L BNN
-F 1 "Jumpper" H 9950 7650 45  0000 L BNN
+F 1 "~" H 9950 7650 45  0000 L BNN
 F 2 "autoSwitch:SMD-Jummper" H 9500 7600 20  0001 C CNN
 F 3 "" H 9650 7650 60  0000 C CNN
@@
 P 9650 7550
 F 0 "JP4" H 9800 7600 45  0000 L BNN
-F 1 "Jumpper" H 9950 7550 45  0000 L BNN
+F 1 "~" H 9950 7550 45  0000 L BNN
 F 2 "autoSwitch:SMD-Jummper" H 9500 7500 20  0001 C CNN
 F 3 "" H 9650 7550 60  0000 C CNN
@@
 P 9650 6650
 F 0 "JP5" H 9800 6700 45  0000 L BNN
-F 1 "Jumpper" H 9950 6650 45  0000 L BNN
+F 1 "~" H 9950 6650 45  0000 L BNN
 F 2 "autoSwitch:SMD-Jummper" H 9500 6600 20  0001 C CNN
 F 3 "" H 9650 6650 60  0000 C CNN
@@
 P 9650 6550
 F 0 "JP6" H 9800 6600 45  0000 L BNN
-F 1 "Jumpper" H 9950 6550 45  0000 L BNN
+F 1 "~" H 9950 6550 45  0000 L BNN
 F 2 "autoSwitch:SMD-Jummper" H 9500 6500 20  0001 C CNN
 F 3 "" H 9650 6550 60  0000 C CNN
@@
 NoConn ~ 12850 7100
 NoConn ~ 12450 6450
+Wire Wire Line
+	6000 9850 6400 9850
+$Comp
+L 0005_064R_1K___CAY16-102J4LF RP1
+U 1 1 5A38C700
+P 10600 6150
+F 0 "RP1" H 10501 6030 70  0000 L BNN
+F 1 "1K" H 10501 5930 70  0000 L BNN
+F 2 "CAY16" H 10590 5940 65  0001 L TNN
+F 3 "" H 10600 6150 60  0001 C CNN
+	1    10600 6150
+	-1   0    0    1
+$EndComp
 $EndSCHEMATC

Commit message: updated Q1 footprint and updated routing
Parts:
- Q1: value BC237 -> s9014; footprint Pin_Headers:Pin_Header_Straight_1x03_Pitch1.27mm -> TO_SOT_Packages_SMD:SOT-23
Changed lines of the file:
@@
 P 12200 6250
 F 0 "Q1" H 12400 6325 50  0000 L CNN
-F 1 "BC237" H 12400 6250 50  0000 L CNN
-F 2 "Pin_Headers:Pin_Header_Straight_1x03_Pitch1.27mm" H 12400 6175 50  0000 L CIN
+F 1 "s9014" H 12400 6250 50  0000 L CNN
+F 2 "TO_SOT_Packages_SMD:SOT-23" H 12400 6175 50  0000 L CIN
 F 3 "" H 12200 6250 50  0000 L CNN
 	1    12200 6250

Commit message: update of routing to move the 4.7uf under the CPU
Parts:
- removed P1: TTL, Pin_Headers:Pin_Header_Straight_1x03, symbol CONN_01X03
- added C2: 100nF, C0603-ROUND, symbol 0015_100NF_0603
- added P1: TTL, Pin_Headers:Pin_Header_Straight_1x04, symbol CONN_01X04
- RL1: value relay -> ~
Connections:
- wire segments 85 -> 87
Changed lines of the file:
@@
 NoConn ~ 9100 6950
 NoConn ~ 9100 6850
-$Comp
-L CONN_01X03 P1
-U 1 1 5A39460E
-P 11200 8250
-F 0 "P1" H 11200 8450 50  0000 C CNN
-F 1 "TTL" V 11300 8250 50  0000 C CNN
-F 2 "Pin_Headers:Pin_Header_Straight_1x03" H 11200 8250 50  0001 C CNN
-F 3 "" H 11200 8250 50  0000 C CNN
-	1    11200 8250
-	1    0    0    -1
-$EndComp
-Text Label 10500 8450 0    65   ~ 0
+Text Label 10500 8350 0    65   ~ 0
 RX
 $Comp
@@
 P 12500 6800
 F 0 "RL1" H 12950 6950 50  0000 L CNN
-F 1 "relay" H 12950 6850 50  0000 L CNN
+F 1 "~" H 12950 6850 50  0000 L CNN
 F 2 "autoSwitch:Relay_HK4100F" H 12500 6800 50  0000 C CNN
 F 3 "" H 12500 6800 50  0000 C CNN
@@
 	1    0    0    -1
 $EndComp
-Wire Wire Line
-	6400 9750 6400 9950
-Wire Wire Line
-	6000 9950 6100 9950
-Wire Wire Line
-	6100 9950 6100 9850
-Connection ~ 6400 9850
-Connection ~ 6100 9850
-Wire Wire Line
-	5700 7550 7200 7550
-Wire Wire Line
-	7200 6950 6700 6950
-Wire Wire Line
-	6700 6950 6700 7650
-Wire Wire Line
-	6200 7650 6200 7850
-Wire Wire Line
-	5100 7650 6200 7650
-Wire Wire Line
-	6700 7650 7200 7650
-Wire Wire Line
-	5100 7650 5100 7750
-Connection ~ 6700 7550
-Connection ~ 5700 7550
-Connection ~ 5700 7650
-Wire Wire Line
-	12700 9750 13000 9750
-Wire Wire Line
-	13000 9750 13000 9550
-Wire Wire Line
-	7200 6850 5000 6850
-Wire Wire Line
-	5000 6850 5000 7050
-Wire Wire Line
-	5000 7350 5000 7450
-Wire Wire Line
-	6200 8150 6200 8350
-Wire Wire Line
-	5700 8150 5700 8250
-Wire Wire Line
-	5100 8250 6200 8250
-Wire Wire Line
-	5100 8250 5100 8050
-Connection ~ 6200 8250
-Connection ~ 5700 8250
-Wire Wire Line
-	12700 9950 13000 9950
-Wire Wire Line
-	13000 9950 13000 10150
-Wire Wire Line
-	5600 10550 5600 10250
-Wire Wire Line
-	11100 6850 11100 6750
-Wire Wire Line
-	6300 6550 6100 6550
-Wire Wire Line
-	6100 6550 6100 6650
-Wire Wire Line
-	7200 7050 7000 7050
-Wire Wire Line
-	7000 7050 7000 7450
-Wire Wire Line
-	6800 7350 7200 7350
-Wire Wire Line
-	7000 7450 7200 7450
-Connection ~ 7000 7350
-Wire Wire Line
-	6400 10450 6400 10250
-Wire Wire Line
-	9100 8250 9900 8250
-Wire Wire Line
-	9100 8150 9900 8150
-Wire Wire Line
-	13600 9850 12700 9850
-Wire Wire Line
-	9100 6350 9500 6350
-Wire Wire Line
-	11400 9750 12400 9750
-Wire Wire Line
-	9100 6250 9500 6250
-Wire Wire Line
-	11400 9850 12400 9850
-Wire Wire Line
-	6900 6450 6600 6450
-Wire Wire Line
-	7200 6550 6900 6550
-Wire Wire Line
-	6900 6550 6900 6450
-Wire Wire Line
-	6600 6650 7200 6650
-Wire Wire Line
-	11100 6150 11100 6450
-Wire Wire Line
-	10800 6150 11100 6150
-Wire Wire Line
-	11400 9950 12400 9950
-Wire Wire Line
-	10300 8150 11000 8150
-Wire Wire Line
-	4800 9750 4800 9850
-Wire Wire Line
-	4800 9850 5300 9850
-Wire Wire Line
-	9100 6150 10400 6150
-Wire Wire Line
-	9900 8250 9900 8350
-Wire Wire Line
-	10300 8350 10700 8350
-Wire Wire Line
-	10700 8350 10700 8250
-Wire Wire Line
-	10700 8250 11000 8250
-Wire Wire Line
-	5700 7250 5700 7850
-Wire Wire Line
-	12300 7100 12300 7200
-Wire Wire Line
-	12300 6500 12300 6450
-Wire Wire Line
-	12300 6000 12300 6050
-Wire Wire Line
-	12000 6250 11750 6250
-Wire Wire Line
-	12600 6500 12600 6400
 $Comp
 L VIN #M016
@@
 	1    0    0    -1
 $EndComp
-Wire Wire Line
-	12600 6400 13450 6400
 $Comp
 L CONN_01X02 P2
@@
 	1    0    0    -1
 $EndComp
-Wire Wire Line
-	12700 7100 12700 7200
-Wire Wire Line
-	12700 7200 13300 7200
 $Comp
 L COM #M017
@@
 	1    0    0    -1
 $EndComp
-Wire Wire Line
-	13300 7450 13300 7300
 Text Label 11800 6250 0    60   ~ 0
 D2
-Wire Wire Line
-	9100 8050 9300 8050
 Text Label 9200 8050 0    60   ~ 0
 D2
@@
 	1    0    0    -1
 $EndComp
-Wire Wire Line
-	9100 6550 9400 6550
-Wire Wire Line
-	9100 6650 9400 6650
-Wire Wire Line
-	9100 7550 9400 7550
-Wire Wire Line
-	9100 7650 9400 7650
-Wire Wire Line
-	9100 7750 9400 7750
-Wire Wire Line
-	9100 7850 9400 7850
-Wire Wire Line
-	9900 6550 10000 6550
-Wire Wire Line
-	10000 6550 10000 7950
-Wire Wire Line
-	10000 7950 9100 7950
-Wire Wire Line
-	9900 7850 10000 7850
-Connection ~ 10000 7850
-Wire Wire Line
-	9900 7750 10000 7750
-Connection ~ 10000 7750
-Wire Wire Line
-	9900 7650 10000 7650
-Connection ~ 10000 7650
-Wire Wire Line
-	9900 7550 10000 7550
-Connection ~ 10000 7550
-Wire Wire Line
-	9900 6650 10000 6650
-Connection ~ 10000 6650
 $Comp
 L CONN_01X02 P3
@@
 	1    0    0    -1
 $EndComp
-Wire Wire Line
-	8500 9700 8500 9850
-Wire Wire Line
-	8500 9850 8600 9850
-Wire Wire Line
-	8600 9950 8500 9950
-Wire Wire Line
-	8500 9950 8500 10050
-Wire Wire Line
-	6200 6150 7200 6150
-Wire Wire Line
-	6200 6150 6200 5950
-Wire Wire Line
-	6200 5550 6200 5450
 Text Label 6200 5950 3    10   ~ 0
 RESET
@@
 NoConn ~ 12850 7100
 NoConn ~ 12450 6450
-Wire Wire Line
-	6000 9850 6400 9850
 $Comp
 L 0005_064R_1K___CAY16-102J4LF RP1
@@
 	-1   0    0    1
 $EndComp
+$Comp
+L CONN_01X04 P1
+U 1 1 5A3EFC05
+P 11200 8200
+F 0 "P1" H 11200 8450 50  0000 C CNN
+F 1 "TTL" V 11300 8200 50  0000 C CNN
+F 2 "Pin_Headers:Pin_Header_Straight_1x04" H 11200 8200 50  0000 C CNN
+F 3 "" H 11200 8200 50  0000 C CNN
+	1    11200 8200
+	1    0    0    -1
+$EndComp
+Text Label 10400 7750 0    60   ~ 0
+RESET
+$Comp
+L 0015_100NF_0603 C2
+U 1 1 5A3F027E
+P 10700 7850
+F 0 "C2" H 10760 7865 45  0000 L BNN
+F 1 "100nF" H 10760 7665 45  0000 L BNN
+F 2 "C0603-ROUND" H 10730 8000 20  0001 C CNN
+F 3 "" H 10700 7850 60  0000 C CNN
+	1    10700 7850
+	1    0    0    -1
+$EndComp
+Wire Wire Line
+	6400 9750 6400 9950
+Wire Wire Line
+	6000 9950 6100 9950
+Wire Wire Line
+	6100 9950 6100 9850
+Connection ~ 6400 9850
+Connection ~ 6100 9850
+Wire Wire Line
+	5700 7550 7200 7550
+Wire Wire Line
+	7200 6950 6700 6950
+Wire Wire Line
+	6700 6950 6700 7650
+Wire Wire Line
+	6200 7650 6200 7850
+Wire Wire Line
+	5100 7650 6200 7650
+Wire Wire Line
+	6700 7650 7200 7650
+Wire Wire Line
+	5100 7650 5100 7750
+Connection ~ 6700 7550
+Connection ~ 5700 7550
+Connection ~ 5700 7650
+Wire Wire Line
+	12700 9750 13000 9750
+Wire Wire Line
+	13000 9750 13000 9550
+Wire Wire Line
+	7200 6850 5000 6850
+Wire Wire Line
+	5000 6850 5000 7050
+Wire Wire Line
+	5000 7350 5000 7450
+Wire Wire Line
+	6200 8150 6200 8350
+Wire Wire Line
+	5700 8150 5700 8250
+Wire Wire Line
+	5100 8250 6200 8250
+Wire Wire Line
+	5100 8250 5100 8050
+Connection ~ 6200 8250
+Connection ~ 5700 8250
+Wire Wire Line
+	12700 9950 13000 9950
+Wire Wire Line
+	13000 9950 13000 10150
+Wire Wire Line
+	5600 10550 5600 10250
+Wire Wire Line
+	11100 6850 11100 6750
+Wire Wire Line
+	6300 6550 6100 6550
+Wire Wire Line
+	6100 6550 6100 6650
+Wire Wire Line
+	7200 7050 7000 7050
+Wire Wire Line
+	7000 7050 7000 7450
+Wire Wire Line
+	6800 7350 7200 7350
+Wire Wire Line
+	7000 7450 7200 7450
+Connection ~ 7000 7350
+Wire Wire Line
+	6400 10450 6400 10250
+Wire Wire Line
+	9100 8250 9900 8250
+Wire Wire Line
+	9100 8150 9900 8150
+Wire Wire Line
+	13600 9850 12700 9850
+Wire Wire Line
+	9100 6350 9500 6350
+Wire Wire Line
+	11400 9750 12400 9750
+Wire Wire Line
+	9100 6250 9500 6250
+Wire Wire Line
+	11400 9850 12400 9850
+Wire Wire Line
+	6900 6450 6600 6450
+Wire Wire Line
+	7200 6550 6900 6550
+Wire Wire Line
+	6900 6550 6900 6450
+Wire Wire Line
+	6600 6650 7200 6650
+Wire Wire Line
+	11100 6150 11100 6450
+Wire Wire Line
+	10800 6150 11100 6150
+Wire Wire Line
+	11400 9950 12400 9950
+Wire Wire Line
+	4800 9750 4800 9850
+Wire Wire Line
+	4800 9850 5300 9850
+Wire Wire Line
+	9100 6150 10400 6150
+Wire Wire Line
+	9900 8250 9900 8350
+Wire Wire Line
+	5700 7250 5700 7850
+Wire Wire Line
+	12300 7100 12300 7200
+Wire Wire Line
+	12300 6500 12300 6450
+Wire Wire Line
+	12300 6000 12300 6050
+Wire Wire Line
+	12000 6250 11750 6250
+Wire Wire Line
+	12600 6500 12600 6400
+Wire Wire Line
+	12600 6400 13450 6400
+Wire Wire Line
+	12700 7100 12700 7200
+Wire Wire Line
+	12700 7200 13300 7200
+Wire Wire Line
+	13300 7450 13300 7300
+Wire Wire Line
+	9100 8050 9300 8050
+Wire Wire Line
+	9100 6550 9400 6550
+Wire Wire Line
+	9100 6650 9400 6650
+Wire Wire Line
+	9100 7550 9400 7550
+Wire Wire Line
+	9100 7650 9400 7650
+Wire Wire Line
+	9100 7750 9400 7750
+Wire Wire Line
+	9100 7850 9400 7850
+Wire Wire Line
+	9900 6550 10000 6550
+Wire Wire Line
+	10000 6550 10000 7950
+Wire Wire Line
+	10000 7950 9100 7950
+Wire Wire Line
+	9900 7850 10000 7850
+Connection ~ 10000 7850
+Wire Wire Line
+	9900 7750 10000 7750
+Connection ~ 10000 7750
+Wire Wire Line
+	9900 7650 10000 7650
+Connection ~ 10000 7650
+Wire Wire Line
+	9900 7550 10000 7550
+Connection ~ 10000 7550
+Wire Wire Line
+	9900 6650 10000 6650
+Connection ~ 10000 6650
+Wire Wire Line
+	8500 9700 8500 9850
+Wire Wire Line
+	8500 9850 8600 9850
+Wire Wire Line
+	8600 9950 8500 9950
+Wire Wire Line
+	8500 9950 8500 10050
+Wire Wire Line
+	6200 6150 7200 6150
+Wire Wire Line
+	6200 6150 6200 5950
+Wire Wire Line
+	6200 5550 6200 5450
+Wire Wire Line
+	6000 9850 6400 9850
+Wire Wire Line
+	10700 8050 11000 8050
+Wire Wire Line
+	10400 7750 10700 7750
+Wire Wire Line
+	10300 8150 11000 8150
+Wire Wire Line
+	10300 8350 10700 8350
+Wire Wire Line
+	10700 8350 10700 8250
+Wire Wire Line
+	10700 8250 11000 8250
 $EndSCHEMATC

Commit message: fixed a footprint error for HK4001 relay
Connections:
- wire segments 87 -> 88
- no-connect marks 12 -> 10
Changed lines of the file:
@@
 	1    0    0    -1
 $EndComp
-NoConn ~ 12800 6500
 $Comp
 L Jumpper JP1
@@
 	0    -1   -1   0
 $EndComp
-NoConn ~ 12850 7100
-NoConn ~ 12450 6450
 $Comp
 L 0005_064R_1K___CAY16-102J4LF RP1
@@
 	12000 6250 11750 6250
 Wire Wire Line
-	12600 6500 12600 6400
-Wire Wire Line
-	12600 6400 13450 6400
-Wire Wire Line
 	12700 7100 12700 7200
 Wire Wire Line
@@
 Wire Wire Line
 	10700 8250 11000 8250
+Wire Wire Line
+	12600 6400 13450 6400
+NoConn ~ 12800 6500
+Wire Wire Line
+	12600 6500 12600 6400
+Wire Wire Line
+	12850 7100 12850 7200
+Connection ~ 12850 7200
 $EndSCHEMATC

Commit message: fixed a bug with the transistor
Parts:
- removed Q1: s9014, TO_SOT_Packages_SMD:SOT-23, symbol BC237
- added Q1: SS8050, TO_SOT_Packages_SMD:SOT-23, symbol SS8050
Changed lines of the file:
@@
 $EndComp
 $Comp
-L COM #U$01
+L COM #U$13
 U 1 1 5A38CCDC
 P 13000 10250
-F 0 "#U$01" H 13050 10300 60  0001 C CNN
+F 0 "#U$13" H 13050 10300 60  0001 C CNN
 F 1 "~" H 13000 10250 60  0001 C CNN
 F 2 "" H 13000 10250 60  0001 C CNN
@@
 $EndComp
 $Comp
-L COM #U$02
+L COM #U$2
 U 1 1 5A38D060
 P 5000 7550
-F 0 "#U$02" H 5050 7600 60  0001 C CNN
+F 0 "#U$2" H 5050 7600 60  0001 C CNN
 F 1 "~" H 5000 7550 60  0001 C CNN
 F 2 "" H 5000 7550 60  0001 C CNN
@@
 $EndComp
 $Comp
-L +5V #U$03
+L +5V #U$12
 U 1 1 5A38D128
 P 13000 9450
-F 0 "#U$03" H 12900 9550 70  0001 L BNN
+F 0 "#U$12" H 12900 9550 70  0001 L BNN
 F 1 "+5V" H 12900 9550 70  0000 L BNN
 F 2 "" H 13000 9450 60  0001 C CNN
@@
 $EndComp
 $Comp
-L COM #U$04
+L COM #U$5
 U 1 1 5A38D18C
 P 6100 6750
-F 0 "#U$04" H 6150 6800 60  0001 C CNN
+F 0 "#U$5" H 6150 6800 60  0001 C CNN
 F 1 "~" H 6100 6750 60  0001 C CNN
 F 2 "" H 6100 6750 60  0001 C CNN
@@
 $EndComp
 $Comp
-L COM #U$05
+L COM #U$7
 U 1 1 5A38D2B8
 P 6200 8450
-F 0 "#U$05" H 6250 8500 60  0001 C CNN
+F 0 "#U$7" H 6250 8500 60  0001 C CNN
 F 1 "~" H 6200 8450 60  0001 C CNN
 F 2 "" H 6200 8450 60  0001 C CNN
@@
 $EndComp
 $Comp
-L +5V #U$06
+L +5V #U$8
 U 1 1 5A38D380
 P 6400 9650
-F 0 "#U$06" H 6300 9750 70  0001 L BNN
+F 0 "#U$8" H 6300 9750 70  0001 L BNN
 F 1 "+5V" H 6300 9750 70  0000 L BNN
 F 2 "" H 6400 9650 60  0001 C CNN
@@
 $EndComp
 $Comp
-L VIN #U$07
+L VIN #U$1
 U 1 1 5A38D3E4
 P 4800 9650
-F 0 "#U$07" H 4720 9750 70  0001 L BNN
+F 0 "#U$1" H 4720 9750 70  0001 L BNN
 F 1 "VIN" H 4720 9750 70  0000 L BNN
 F 2 "" H 4800 9650 60  0001 C CNN
@@
 $EndComp
 $Comp
-L COM #U$08
+L COM #U$9
 U 1 1 5A38D448
 P 6400 10550
-F 0 "#U$08" H 6450 10600 60  0001 C CNN
+F 0 "#U$9" H 6450 10600 60  0001 C CNN
 F 1 "~" H 6400 10550 60  0001 C CNN
 F 2 "" H 6400 10550 60  0001 C CNN
@@
 $EndComp
 $Comp
-L COM #U$09
+L COM #U$3
 U 1 1 5A38D8F8
 P 5600 10650
-F 0 "#U$09" H 5650 10700 60  0001 C CNN
+F 0 "#U$3" H 5650 10700 60  0001 C CNN
 F 1 "~" H 5600 10650 60  0001 C CNN
 F 2 "" H 5600 10650 60  0001 C CNN
@@
 $EndComp
 $Comp
-L COM #U$010
+L COM #U$11
 U 1 1 5A38D95C
 P 11100 6950
-F 0 "#U$010" H 11150 7000 60  0001 C CNN
+F 0 "#U$11" H 11150 7000 60  0001 C CNN
 F 1 "~" H 11100 6950 60  0001 C CNN
 F 2 "" H 11100 6950 60  0001 C CNN
@@
 $EndComp
 $Comp
-L COM #U$011
+L COM #U$10
 U 1 1 5A38DAEC
 P 6800 7450
-F 0 "#U$011" H 6850 7500 60  0001 C CNN
+F 0 "#U$10" H 6850 7500 60  0001 C CNN
 F 1 "~" H 6800 7450 60  0001 C CNN
 F 2 "" H 6800 7450 60  0001 C CNN
@@
 $EndComp
 $Comp
-L +5V #U$012
+L +5V #U$4
 U 1 1 5A38DCE0
 P 5700 7150
-F 0 "#U$012" H 5600 7250 70  0001 L BNN
+F 0 "#U$4" H 5600 7250 70  0001 L BNN
 F 1 "+5V" H 5600 7250 70  0000 L BNN
 F 2 "" H 5700 7150 60  0001 C CNN
@@
 RX
 $Comp
-L COM #M013
+L COM #M3
 U 1 1 5A394983
 P 11000 8450
-F 0 "#M013" H 11000 8450 45  0001 C CNN
+F 0 "#M3" H 11000 8450 45  0001 C CNN
 F 1 "COM" H 11000 8450 45  0001 C CNN
 F 2 "" H 11000 8450 60  0000 C CNN
@@
 $EndComp
 $Comp
-L COM #M014
+L COM #M5
 U 1 1 5A3B4697
 P 12300 7300
-F 0 "#M014" H 12300 7300 45  0001 C CNN
+F 0 "#M5" H 12300 7300 45  0001 C CNN
 F 1 "COM" H 12300 7300 45  0001 C CNN
 F 2 "" H 12300 7300 60  0000 C CNN
@@
 $EndComp
 $Comp
-L +5V #M015
+L +5V #M4
 U 1 1 5A3B46CD
 P 12300 5900
-F 0 "#M015" H 12300 5900 45  0001 L BNN
+F 0 "#M4" H 12300 5900 45  0001 L BNN
 F 1 "+5V" H 12200 6000 45  0000 L BNN
 F 2 "" H 12300 5900 60  0000 C CNN
@@
 $EndComp
 $Comp
-L BC237 Q1
-U 1 1 5A3B4AFF
-P 12200 6250
-F 0 "Q1" H 12400 6325 50  0000 L CNN
-F 1 "s9014" H 12400 6250 50  0000 L CNN
-F 2 "TO_SOT_Packages_SMD:SOT-23" H 12400 6175 50  0000 L CIN
-F 3 "" H 12200 6250 50  0000 L CNN
-	1    12200 6250
-	1    0    0    -1
-$EndComp
-$Comp
-L VIN #M016
+L VIN #M7
 U 1 1 5A3B5FE9
 P 13450 6300
-F 0 "#M016" H 13450 6300 45  0001 L BNN
+F 0 "#M7" H 13450 6300 45  0001 L BNN
 F 1 "VIN" H 13370 6400 45  0000 L BNN
 F 2 "" H 13450 6300 60  0000 C CNN
@@
 $EndComp
 $Comp
-L COM #M017
+L COM #M6
 U 1 1 5A3B62DB
 P 13300 7550
-F 0 "#M017" H 13300 7550 45  0001 C CNN
+F 0 "#M6" H 13300 7550 45  0001 C CNN
 F 1 "COM" H 13300 7550 45  0001 C CNN
 F 2 "" H 13300 7550 60  0000 C CNN
@@
 $EndComp
 $Comp
-L VIN #M018
+L VIN #M1
 U 1 1 5A3B8248
 P 8500 9600
-F 0 "#M018" H 8500 9600 45  0001 L BNN
+F 0 "#M1" H 8500 9600 45  0001 L BNN
 F 1 "VIN" H 8420 9700 45  0000 L BNN
 F 2 "" H 8500 9600 60  0000 C CNN
@@
 $EndComp
 $Comp
-L COM #M019
+L COM #M2
 U 1 1 5A3B8290
 P 8500 10150
-F 0 "#M019" H 8500 10150 45  0001 C CNN
+F 0 "#M2" H 8500 10150 45  0001 C CNN
 F 1 "COM" H 8500 10150 45  0001 C CNN
 F 2 "" H 8500 10150 60  0000 C CNN
@@
 +5V
 $Comp
-L +5V #U$020
+L +5V #U$6
 U 1 1 5A38D894
 P 6200 5350
-F 0 "#U$020" H 6100 5450 70  0001 L BNN
+F 0 "#U$6" H 6100 5450 70  0001 L BNN
 F 1 "+5V" H 6100 5450 70  0000 L BNN
 F 2 "" H 6200 5350 60  0001 C CNN
@@
 	12850 7100 12850 7200
 Connection ~ 12850 7200
+$Comp
+L SS8050 Q1
+U 1 1 5A4605D3
+P 12200 6250
+F 0 "Q1" H 12400 6325 50  0000 L CNN
+F 1 "SS8050" H 12400 6250 50  0000 L CNN
+F 2 "TO_SOT_Packages_SMD:SOT-23" H 12400 6175 50  0000 L CIN
+F 3 "" H 12200 6250 50  0000 L CNN
+	1    12200 6250
+	1    0    0    -1
+$EndComp
 $EndSCHEMATC
