File: kicad/NanoV3.2.kicad_pcb (KiCad board)
At the start: 2 copper layers, 43.2 x 17.8 mm, 23 parts, among them IC2 LM1117, IC3 ATMEGA328P-AU, P1 TTL, P2 OUT, P3 INPUT, Q1 BC237, Y1 16MHz

Commit message: finished layout
Routing:
- net Net-(P2-Pad1): track 4.84 -> 10.4 mm
Other:
- net class w1.0 added: clearance 0.4, trace_width 1, via_dia 2.4, via_drill 1.6
Changed lines of the file:
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@@
     (thickness 1.6)
     (drawings 89)
-    (tracks 276)
+    (tracks 278)
     (zones 0)
     (modules 23)
@@
     (34 B.Paste user)
     (35 F.Paste user)
-    (36 B.SilkS user hide)
-    (37 F.SilkS user hide)
-    (38 B.Mask user hide)
-    (39 F.Mask user hide)
-    (40 Dwgs.User user hide)
+    (36 B.SilkS user)
+    (37 F.SilkS user)
+    (38 B.Mask user)
+    (39 F.Mask user)
+    (40 Dwgs.User user)
     (41 Cmts.User user)
     (42 Eco1.User user)
-    (43 Eco2.User user hide)
+    (43 Eco2.User user)
     (44 Edge.Cuts user)
     (45 Margin user)
@@
     (visible_elements 7FFFFFFF)
     (pcbplotparams
-      (layerselection 0x00030_80000001)
+      (layerselection 0x3ffff_80000001)
       (usegerberextensions false)
       (excludeedgelayer true)
@@
       (outputformat 1)
       (mirror false)
-      (drillshape 1)
+      (drillshape 0)
       (scaleselection 1)
-      (outputdirectory ""))
+      (outputdirectory outputs/))
   )
   (net 0 "")
@@
     (add_net COM)
     (add_net "Net-(P1-Pad2)")
-    (add_net "Net-(P2-Pad1)")
     (add_net "Net-(Q1-Pad3)")
-    (add_net VIN)
   )
   (net_class w0.5 ""
@@
     (uvia_dia 0.6)
     (uvia_drill 0.2)
+  )
+  (net_class w1.0 ""
+    (clearance 0.4)
+    (trace_width 1)
+    (via_dia 2.4)
+    (via_drill 1.6)
+    (uvia_dia 1.2)
+    (uvia_drill 0.4)
+    (add_net "Net-(P2-Pad1)")
+    (add_net VIN)
   )
   (module 2X03 (layer Top)
@@
       (effects (font (size 0.57912 0.57912) (thickness 0.046329)) (justify left bottom))
     )
-    (fp_text value 1uF (at -0.889 2.032 405) (layer F.SilkS)
+    (fp_text value 1uF (at 0.434644 -2.130117 405) (layer F.SilkS)
       (effects (font (size 0.57912 0.57912) (thickness 0.046329)) (justify left bottom))
     )
@@
   (segment (start 141.65072 106.82224) (end 141.645 106.82796) (width 0.25) (layer Top) (net 14))
   (segment (start 141.645 106.82796) (end 141.645 107.512) (width 0.25) (layer Top) (net 14))
-  (segment (start 155.88488 111.14532) (end 157.69336 111.14532) (width 0.25) (layer Bottom) (net 15))
-  (segment (start 162.55492 106.28376) (end 167.52824 106.28376) (width 0.25) (layer Bottom) (net 15))
-  (segment (start 157.69336 111.14532) (end 162.55492 106.28376) (width 0.25) (layer Bottom) (net 15))
+  (segment (start 155.88488 111.14532) (end 157.2768 111.14532) (width 1) (layer Bottom) (net 15) (status 400000))
+  (segment (start 162.13836 106.28376) (end 167.52824 106.28376) (width 1) (layer Bottom) (net 15) (status 800000))
+  (segment (start 157.2768 111.14532) (end 162.13836 106.28376) (width 1) (layer Bottom) (net 15))
   (segment (start 150.2918 103.0986) (end 152.13076 103.0986) (width 0.25) (layer Top) (net 15))
   (segment (start 154.2288 109.48924) (end 155.88488 111.14532) (width 0.25) (layer Top) (net 15))
@@
   (segment (start 151.31288 110.998) (end 150.65248 111.6584) (width 0.25) (layer Bottom) (net 23))
   (segment (start 138.365226 106.544106) (end 138.365226 106.465428) (width 0.25) (layer Top) (net 23))
-  (segment (start 163.50488 98.44532) (end 165.5572 98.44532) (width 0.25) (layer Bottom) (net 24))
+  (segment (start 163.50488 98.44532) (end 165.5572 98.44532) (width 1) (layer Bottom) (net 24) (status 400000))
+  (segment (start 165.5572 98.44532) (end 167.52824 100.41636) (width 1) (layer Bottom) (net 24) (status 800000))
+  (segment (start 165.5572 98.44532) (end 167.52824 100.41636) (width 0.5) (layer Bottom) (net 24))
   (segment (start 165.5572 98.44532) (end 167.52824 100.41636) (width 0.25) (layer Bottom) (net 24))
   (segment (start 152.273 109.728) (end 154.7622 109.728) (width 0.25) (layer Bottom) (net 25))
